Commit message: Put together all the pieces to successfully run project to default map

File: urdf/udacity_bot_sebastian.xacro (robot description, xacro)
@@ -175,4 +175,13 @@
     <parent link="chassis"/>
   </joint>
+  <!-- OPTICAL FRAME: Workaround needed so depth cloud points in the right direction -->
+  <joint name="camera_optical_joint" type="fixed">
+    <origin xyz="0 0 0" rpy="${-pi/2} 0 ${-pi/2}"/>
+    <parent link="camera"/>
+    <child link="camera_link_optical"/>
+  </joint>
+  <link name="camera_link_optical">
+  </link>
+  <!-- END OPTICAL FRAME -->
   <!-- LIDAR -->
     <link name='lidar_mount'>
